File: design/schematics/PayloadBay.sch (EAGLE design)
At the start: 72 parts, among them IC1 MC33269ST-5.0T3, IC2 MC33269D-5.0, IC3 ATMEGA2560-16AU, IC4 ATMEGA8U2-MU, IC5 LM358D, IC6 LP2985-33DBVR, Q1 16MHz, Q2 16MHz, T2 FDN340P, X1 DC21MMX, Y1 16MHz, Y2 16MHz

Commit message: updated schematics and board
* also added backup files made by eagle to gitignore
Parts:
- removed ADCH, ADCL, COMMUNICATION, PWMH, PWML: (no value), pinhead:PINHD-1X8
- removed C10: 1u, SmartPrj:C-EU0603-RND
- removed C11, C8: 100n, rcl:C-EUC0603
- removed C12, C13, C7, C9: 100n, SmartPrj:C-EU0603-RND
- removed C16, C17: 22p, SmartPrj:C-EU0603-RND
- removed F1: 500mA, rcl:L-EUL1812
- removed GROUND, RESET-EN, UBOOT: (no value), jumper:SJ
- removed IC4: ATMEGA8U2-MU, atmel:ATMEGA8U2-MU
- removed IC5: LM358D, linear:LM358D
- removed IC6: LP2985-33DBVR, texas:TPS77033
- removed ICSP1: ICSP, pinhead:PINHD-2X3
- removed JP1, JP2, JP3, JP4: (no value), pinhead:PINHD-1X1
- removed L1: BLM21, wuerth-elektronik:WE-CBF_0805
- removed POWER: (no value), pinhead:PINHD-1X6
- removed Q1: 16MHz, special:XTAL/S
- removed R2: 1M, SmartPrj:R-EU_R0603
- removed R4: 27R, SmartPrj:R-EU_R0603
- removed RN2: 22R, resistor-dil:4R-NCAY16
- removed RN4: 1k, resistor-dil:4R-NCAY16
- removed RN5: 10K, resistor-dil:4R-NCAT16
- removed RX, TX: YELLOW, led:LEDCHIP-LED0805
- removed T2: FDN340P, zetex:PMOSSOT23
- removed U$2, U$3, U$4, U$5: FIDUCIALMOUNT, SmartPrj:FIDUCIALMOUNT
- removed X2: (no value), SmartPrj:PN61729
- removed XIOH, XIOL: (no value), pinhead:PINHD-2X8
- removed Y2: 16MHz, SmartPrj:RESONATORMU
- removed Z1, Z2: PGB1010604, varistor:VARISTORCN0603
Connections:
- removed net +3V3: C13.2, IC5B.-IN, IC6.OUT, POWER.2
- removed net CMP: C12.2, IC5B.+IN, RN5B.2, RN5C.1
- removed net D+: RN2D.2, X2.3, Z2.2
- removed net D-: RN2A.2, X2.2, Z1.2
- removed net DTR: C7.1, IC4.(CTS/HWB/AIN6/TO/INT7)PD7, UBOOT.1
- removed net GATE_CMD: IC5B.OUT, T2.G
- removed net M8RXD: IC4.(TXD1/INT3)PD3, RN4B.2
- removed net M8TXD: IC4.(RXD1/AIN1/INT2)PD2, RN4A.2
- removed net MISO2: IC4.(PD0/MISO/PCINT3)PB3, ICSP1.1
- removed net MOSI2: IC4.(PDI/MOSI/PCINT2)PB2, ICSP1.4
- removed net N$54: RN4D.1, RX.A
- removed net N$55: RN4C.1, TX.A
- removed net RD+: IC4.D+, RN2D.1
- removed net RD-: IC4.D-, RN2A.1
- removed net RESET2: IC4.RESET(PC1/DW), ICSP1.5, RN5A.2
- removed net RXL: IC4.(INT5/AIN3)PD4, RX.C
- removed net SCK2: IC4.(SCLK/PCINT1)PB1, ICSP1.3
- removed net TXL: IC4.(XCK/AIN4/PCINT12)PD5, TX.C
- removed net UGND: C10.2, GROUND.1, IC4.UGND, L1.1, X2.4
- removed net USBVCC: C8.1, F1.1, IC4.UVCC, T2.D
- removed net USHIELD: L1.2, X2.P$1, X2.P$2, Z1.1, Z2.1
- removed net VUCAP: C10.1, IC4.UCAP
- removed net XT1: C16.1, Q1.2, R2.1, R4.2, Y2.3
- removed net XT1R: IC4.XTAL1, R4.1
- removed net XT2: C17.1, IC4.XTAL2(PC0), Q1.1, R2.2, Y2.1
- removed net XVCC: F1.2, X2.1
- net +5V: no longer C11.2, C9.1, IC4.AVCC, IC4.VCC, IC5P.V+, IC6.!EN, IC6.IN, ICSP1.2, JP1.1, JP2.1, POWER.3, RN4C.2, RN4D.2, RN5A.1, T2.S
- net ADC0: no longer ADCL.1
- net ADC1: no longer ADCL.2
- net ADC10: no longer ADCH.3
- net ADC11: no longer ADCH.4
- net ADC12: no longer ADCH.5
- net ADC13: no longer ADCH.6
- net ADC14: no longer ADCH.7
- net ADC15: no longer ADCH.8
- net ADC2: no longer ADCL.3
- net ADC3: no longer ADCL.4
- net ADC4: no longer ADCL.5
- net ADC5: no longer ADCL.6
- net ADC6: no longer ADCL.7
- net ADC7: no longer ADCL.8
- net ADC8: no longer ADCH.1
- net ADC9: no longer ADCH.2
- net AREF: no longer PWMH.8
- net GND: no longer C11.1, C12.1, C13.1, C16.2, C17.2, C8.2, C9.2, GROUND.2, IC4.GND, IC4.PAD, IC5A.+IN, IC5A.-IN, IC5P.V-, IC6.GND, ICSP1.6, JP3.1, JP4.1, POWER.4, POWER.5, PWMH.7, RN5B.1, UBOOT.2, Y2.2
- net PA0: no longer XIOH.16
- net PA1: no longer XIOH.15
- net PA2: no longer XIOH.14
- net PA3: no longer XIOH.13
- net PA4: no longer XIOH.12
- net PA5: no longer XIOH.11
- net PA6: no longer XIOH.10
- net PA7: no longer XIOH.9
- net PB0: no longer XIOL.1
- net PB1: no longer XIOL.2
- net PB2: no longer XIOL.3
- net PB3: no longer XIOL.4
- net PB4: no longer PWMH.3
- net PB5: no longer PWMH.4
- net PB6: no longer PWMH.5
- net PB7: no longer PWMH.6
- net PC0: no longer XIOH.1
- net PC1: no longer XIOH.2
- net PC2: no longer XIOH.3
- net PC3: no longer XIOH.4
- net PC4: no longer XIOH.5
- net PC5: no longer XIOH.6
- net PC6: no longer XIOH.7
- net PC7: no longer XIOH.8
- net PD7: no longer XIOL.16
- net PE0: no longer PWML.1, RN4B.1
- net PE1: no longer PWML.2, RN4A.1
- net PE3: no longer PWML.6
- net PE4: no longer PWML.3
- net PE5: no longer PWML.4
- net PG0: no longer XIOL.13
- net PG1: no longer XIOL.14
- net PG2: no longer XIOL.15
- net PG5: no longer PWML.5
- net PH3: no longer PWML.7
- net PH4: no longer PWML.8
- net PH5: no longer PWMH.1
- net PH6: no longer PWMH.2
- net PL0: no longer XIOL.5
- net PL1: no longer XIOL.6
- net PL2: no longer XIOL.7
- net PL3: no longer XIOL.8
- net PL4: no longer XIOL.9
- net PL5: no longer XIOL.10
- net PL6: no longer XIOL.11
- net PL7: no longer XIOL.12
- net RESET: no longer C7.2, POWER.1, RESET-EN.1, RESET-EN.2
- net RXD1: no longer COMMUNICATION.3
- net RXD2: no longer COMMUNICATION.5
- net RXD3: no longer COMMUNICATION.7
- net SCL: no longer COMMUNICATION.1
- net SDA: no longer COMMUNICATION.2
- net TXD1: no longer COMMUNICATION.4
- net TXD2: no longer COMMUNICATION.6
- net TXD3: no longer COMMUNICATION.8
- net VIN: no longer POWER.6, RN5C.2
Other:
- note removed: "(SS)"
- note removed: "0"
- note removed: "1"
- note removed: "10"
- note removed: "11"
- note removed: "12"
- note removed: "13"
- note removed: "14"
- note removed: "15"
- note removed: "16"
- note removed: "17"
- note removed: "18"
- note removed: "19"
- note removed: "2"
- note removed: "20"
- note removed: "21"
- note removed: "22"
- note removed: "23"
- note removed: "24"
- note removed: "25"
- note removed: "26"
- note removed: "27"
- note removed: "28"
- note removed: "29"
- note removed: "3"
- note removed: "30"
- note removed: "31"
- note removed: "32"
- note removed: "33"
- note removed: "34"
- note removed: "35"
- note removed: "36"
- note removed: "37"
- note removed: "38"
- note removed: "39"
- note removed: "4"
- note removed: "40"
- note removed: "41"
- note removed: "42"
- note removed: "43"
- note removed: "44"
- note removed: "45"
- note removed: "46"
- note removed: "47"
- note removed: "48"
- note removed: "49"
- note removed: "5"
- note removed: "50"
- note removed: "51"
- note removed: "52"
- note removed: "53"
- note removed: "6"
- note removed: "7"
- note removed: "8"
- note removed: "9"
- note removed: "USB boot En"
- moved on the sheet: C1, C14, C15, ICSP, Q2, RESET, RN1A, RN1B, RN1C, RN1D, RN3A, RN3B
