File: design/schematics/ArmControl/AGSE_BBB_cape.sch (EAGLE design)
At the start: 54 parts, among them Q1 PFET-FQP27P06, Q2 PFET-FQP27P06, Q3 NFET-FQP30N06L, Q4 PFET-FQP27P06, Q5 NFET-FQP30N06L, Q6 PFET-FQP27P06, Q7 NFET-FQP30N06L, Q8 NFET-FQP30N06L, T1 2N2222, T2 2N2222, T3 2N2222, T4 2N2222, T5 2N3904, T6 2N3904, U1 V_REG_LD1085D2

Commit message: updated schematic symbols for h-bridges
Connections:
- net +5V: now also Q1.D, Q6.D; no longer Q1.S, Q6.S
- net GND: now also Q3.S, Q7.S; no longer Q3.D, Q7.D
- net N$1: now also Q1.S, Q3.D; no longer Q1.D, Q3.S
- net N$11: now also Q6.S, Q7.D; no longer Q6.D, Q7.S
Other:
- moved on the sheet: Q1, Q3, Q6, Q7
Changed lines of the file:
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@@
 <instance part="GND9" gate="1" x="180.34" y="-60.96"/>
 <instance part="Q4" gate="G$1" x="165.1" y="-5.08"/>
-<instance part="Q1" gate="G$1" x="198.12" y="-10.16" rot="R180"/>
-<instance part="Q3" gate="G$1" x="198.12" y="-40.64" rot="R180"/>
+<instance part="Q1" gate="G$1" x="198.12" y="-10.16" rot="MR0"/>
+<instance part="Q3" gate="G$1" x="198.12" y="-43.18" rot="MR0"/>
 <instance part="Q5" gate="G$1" x="165.1" y="-38.1"/>
 <instance part="R4" gate="G$1" x="152.4" y="0" rot="R90"/>
@@
 <instance part="GND10" gate="1" x="180.34" y="20.32"/>
 <instance part="Q2" gate="G$1" x="165.1" y="76.2"/>
-<instance part="Q6" gate="G$1" x="198.12" y="71.12" rot="R180"/>
-<instance part="Q7" gate="G$1" x="198.12" y="40.64" rot="R180"/>
+<instance part="Q6" gate="G$1" x="198.12" y="71.12" rot="MR0"/>
+<instance part="Q7" gate="G$1" x="198.12" y="40.64" rot="MR0"/>
 <instance part="Q8" gate="G$1" x="165.1" y="45.72"/>
 <instance part="R8" gate="G$1" x="152.4" y="81.28" rot="R90"/>
@@
 <wire x1="165.1" y1="-43.18" x2="165.1" y2="-58.42" width="0.1524" layer="91"/>
 <wire x1="165.1" y1="-58.42" x2="180.34" y2="-58.42" width="0.1524" layer="91"/>
-<pinref part="Q3" gate="G$1" pin="D"/>
-<wire x1="198.12" y1="-45.72" x2="198.12" y2="-58.42" width="0.1524" layer="91"/>
+<wire x1="210.82" y1="-58.42" x2="198.12" y2="-58.42" width="0.1524" layer="91"/>
+<pinref part="T1" gate="G$1" pin="E"/>
 <wire x1="198.12" y1="-58.42" x2="180.34" y2="-58.42" width="0.1524" layer="91"/>
-<pinref part="T1" gate="G$1" pin="E"/>
 <wire x1="152.4" y1="-55.88" x2="152.4" y2="-58.42" width="0.1524" layer="91"/>
 <wire x1="152.4" y1="-58.42" x2="165.1" y2="-58.42" width="0.1524" layer="91"/>
 <pinref part="T2" gate="G$1" pin="E"/>
 <wire x1="210.82" y1="-55.88" x2="210.82" y2="-58.42" width="0.1524" layer="91"/>
-<wire x1="210.82" y1="-58.42" x2="198.12" y2="-58.42" width="0.1524" layer="91"/>
-<junction x="198.12" y="-58.42"/>
 <junction x="180.34" y="-58.42"/>
 <junction x="165.1" y="-58.42"/>
+<pinref part="Q3" gate="G$1" pin="S"/>
+<wire x1="198.12" y1="-48.26" x2="198.12" y2="-58.42" width="0.1524" layer="91"/>
+<junction x="198.12" y="-58.42"/>
 </segment>
 <segment>
@@
 <wire x1="165.1" y1="40.64" x2="165.1" y2="22.86" width="0.1524" layer="91"/>
 <wire x1="165.1" y1="22.86" x2="180.34" y2="22.86" width="0.1524" layer="91"/>
-<pinref part="Q7" gate="G$1" pin="D"/>
-<wire x1="198.12" y1="35.56" x2="198.12" y2="22.86" width="0.1524" layer="91"/>
+<wire x1="210.82" y1="22.86" x2="198.12" y2="22.86" width="0.1524" layer="91"/>
+<pinref part="T3" gate="G$1" pin="E"/>
 <wire x1="198.12" y1="22.86" x2="180.34" y2="22.86" width="0.1524" layer="91"/>
-<pinref part="T3" gate="G$1" pin="E"/>
 <wire x1="152.4" y1="25.4" x2="152.4" y2="22.86" width="0.1524" layer="91"/>
 <wire x1="152.4" y1="22.86" x2="165.1" y2="22.86" width="0.1524" layer="91"/>
 <pinref part="T4" gate="G$1" pin="E"/>
 <wire x1="210.82" y1="25.4" x2="210.82" y2="22.86" width="0.1524" layer="91"/>
-<wire x1="210.82" y1="22.86" x2="198.12" y2="22.86" width="0.1524" layer="91"/>
-<junction x="198.12" y="22.86"/>
 <junction x="180.34" y="22.86"/>
 <junction x="165.1" y="22.86"/>
+<pinref part="Q7" gate="G$1" pin="S"/>
+<wire x1="198.12" y1="35.56" x2="198.12" y2="22.86" width="0.1524" layer="91"/>
+<junction x="198.12" y="22.86"/>
 </segment>
 <segment>
@@
 <pinref part="P+2" gate="1" pin="+5V"/>
 <wire x1="180.34" y1="5.08" x2="180.34" y2="10.16" width="0.1524" layer="91"/>
-<pinref part="Q1" gate="G$1" pin="S"/>
-<wire x1="198.12" y1="-5.08" x2="198.12" y2="5.08" width="0.1524" layer="91"/>
+<wire x1="210.82" y1="5.08" x2="198.12" y2="5.08" width="0.1524" layer="91"/>
+<pinref part="R4" gate="G$1" pin="2"/>
 <wire x1="198.12" y1="5.08" x2="180.34" y2="5.08" width="0.1524" layer="91"/>
-<pinref part="R4" gate="G$1" pin="2"/>
 <wire x1="165.1" y1="5.08" x2="152.4" y2="5.08" width="0.1524" layer="91"/>
 <pinref part="R5" gate="G$1" pin="2"/>
-<wire x1="198.12" y1="5.08" x2="210.82" y2="5.08" width="0.1524" layer="91"/>
 <junction x="165.1" y="5.08"/>
 <junction x="180.34" y="5.08"/>
+<pinref part="Q1" gate="G$1" pin="D"/>
+<wire x1="198.12" y1="-5.08" x2="198.12" y2="5.08" width="0.1524" layer="91"/>
 <junction x="198.12" y="5.08"/>
 </segment>
@@
 <wire x1="165.1" y1="86.36" x2="180.34" y2="86.36" width="0.1524" layer="91"/>
 <pinref part="P+1" gate="1" pin="+5V"/>
-<pinref part="Q6" gate="G$1" pin="S"/>
-<wire x1="198.12" y1="76.2" x2="198.12" y2="86.36" width="0.1524" layer="91"/>
+<wire x1="210.82" y1="86.36" x2="198.12" y2="86.36" width="0.1524" layer="91"/>
+<pinref part="R8" gate="G$1" pin="2"/>
 <wire x1="198.12" y1="86.36" x2="180.34" y2="86.36" width="0.1524" layer="91"/>
-<pinref part="R8" gate="G$1" pin="2"/>
 <wire x1="165.1" y1="86.36" x2="152.4" y2="86.36" width="0.1524" layer="91"/>
 <pinref part="R9" gate="G$1" pin="2"/>
-<wire x1="198.12" y1="86.36" x2="210.82" y2="86.36" width="0.1524" layer="91"/>
-<junction x="198.12" y="86.36"/>
 <junction x="165.1" y="86.36"/>
 <junction x="180.34" y="86.36"/>
+<pinref part="Q6" gate="G$1" pin="D"/>
+<wire x1="198.12" y1="76.2" x2="198.12" y2="86.36" width="0.1524" layer="91"/>
+<junction x="198.12" y="86.36"/>
 </segment>
 <segment>
@@
 <net name="N$1" class="0">
 <segment>
-<pinref part="Q1" gate="G$1" pin="D"/>
-<pinref part="Q3" gate="G$1" pin="S"/>
-<wire x1="198.12" y1="-15.24" x2="198.12" y2="-17.78" width="0.1524" layer="91"/>
-<wire x1="198.12" y1="-17.78" x2="198.12" y2="-35.56" width="0.1524" layer="91"/>
 <wire x1="180.34" y1="-17.78" x2="198.12" y2="-17.78" width="0.1524" layer="91"/>
-<junction x="198.12" y="-17.78"/>
 <pinref part="Z-AXIS" gate="G$1" pin="2"/>
 <wire x1="180.34" y1="-20.32" x2="180.34" y2="-17.78" width="0.1524" layer="91"/>
+<pinref part="Q3" gate="G$1" pin="D"/>
+<wire x1="198.12" y1="-38.1" x2="198.12" y2="-17.78" width="0.1524" layer="91"/>
+<pinref part="Q1" gate="G$1" pin="S"/>
+<wire x1="198.12" y1="-17.78" x2="198.12" y2="-15.24" width="0.1524" layer="91"/>
+<junction x="198.12" y="-17.78"/>
 </segment>
 </net>
@@
 <segment>
 <pinref part="R5" gate="G$1" pin="1"/>
+<wire x1="210.82" y1="-5.08" x2="210.82" y2="-10.16" width="0.1524" layer="91"/>
+<pinref part="T2" gate="G$1" pin="C"/>
+<pinref part="Q3" gate="G$1" pin="G"/>
+<wire x1="210.82" y1="-10.16" x2="210.82" y2="-43.18" width="0.1524" layer="91"/>
+<wire x1="210.82" y1="-43.18" x2="210.82" y2="-45.72" width="0.1524" layer="91"/>
+<wire x1="205.74" y1="-43.18" x2="210.82" y2="-43.18" width="0.1524" layer="91"/>
 <pinref part="Q1" gate="G$1" pin="G"/>
-<wire x1="210.82" y1="-5.08" x2="210.82" y2="-10.16" width="0.1524" layer="91"/>
-<wire x1="210.82" y1="-10.16" x2="205.74" y2="-10.16" width="0.1524" layer="91"/>
-<pinref part="Q3" gate="G$1" pin="G"/>
-<wire x1="210.82" y1="-10.16" x2="210.82" y2="-40.64" width="0.1524" layer="91"/>
-<wire x1="210.82" y1="-40.64" x2="205.74" y2="-40.64" width="0.1524" layer="91"/>
-<pinref part="T2" gate="G$1" pin="C"/>
-<wire x1="210.82" y1="-40.64" x2="210.82" y2="-45.72" width="0.1524" layer="91"/>
+<wire x1="205.74" y1="-10.16" x2="210.82" y2="-10.16" width="0.1524" layer="91"/>
+<junction x="210.82" y="-43.18"/>
 <junction x="210.82" y="-10.16"/>
-<junction x="210.82" y="-40.64"/>
 </segment>
 </net>
@@
 <net name="N$11" class="0">
 <segment>
-<pinref part="Q6" gate="G$1" pin="D"/>
-<pinref part="Q7" gate="G$1" pin="S"/>
-<wire x1="198.12" y1="66.04" x2="198.12" y2="63.5" width="0.1524" layer="91"/>
-<wire x1="198.12" y1="63.5" x2="198.12" y2="45.72" width="0.1524" layer="91"/>
 <wire x1="180.34" y1="63.5" x2="198.12" y2="63.5" width="0.1524" layer="91"/>
-<junction x="198.12" y="63.5"/>
 <pinref part="R-AXIS" gate="G$1" pin="2"/>
 <wire x1="180.34" y1="60.96" x2="180.34" y2="63.5" width="0.1524" layer="91"/>
+<pinref part="Q6" gate="G$1" pin="S"/>
+<wire x1="198.12" y1="66.04" x2="198.12" y2="63.5" width="0.1524" layer="91"/>
+<pinref part="Q7" gate="G$1" pin="D"/>
+<wire x1="198.12" y1="45.72" x2="198.12" y2="63.5" width="0.1524" layer="91"/>
+<junction x="198.12" y="63.5"/>
 </segment>
 </net>
@@
 <segment>
 <pinref part="R9" gate="G$1" pin="1"/>
+<wire x1="210.82" y1="76.2" x2="210.82" y2="71.12" width="0.1524" layer="91"/>
+<wire x1="210.82" y1="71.12" x2="210.82" y2="40.64" width="0.1524" layer="91"/>
+<pinref part="T4" gate="G$1" pin="C"/>
 <pinref part="Q6" gate="G$1" pin="G"/>
-<wire x1="210.82" y1="76.2" x2="210.82" y2="71.12" width="0.1524" layer="91"/>
-<wire x1="210.82" y1="71.12" x2="205.74" y2="71.12" width="0.1524" layer="91"/>
+<wire x1="210.82" y1="40.64" x2="210.82" y2="35.56" width="0.1524" layer="91"/>
+<wire x1="205.74" y1="71.12" x2="210.82" y2="71.12" width="0.1524" layer="91"/>
+<junction x="210.82" y="71.12"/>
 <pinref part="Q7" gate="G$1" pin="G"/>
-<wire x1="210.82" y1="71.12" x2="210.82" y2="40.64" width="0.1524" layer="91"/>
-<wire x1="210.82" y1="40.64" x2="205.74" y2="40.64" width="0.1524" layer="91"/>
-<pinref part="T4" gate="G$1" pin="C"/>
-<wire x1="210.82" y1="40.64" x2="210.82" y2="35.56" width="0.1524" layer="91"/>
-<junction x="210.82" y="71.12"/>
+<wire x1="205.74" y1="40.64" x2="210.82" y2="40.64" width="0.1524" layer="91"/>
 <junction x="210.82" y="40.64"/>
 </segment>

Commit message: fixed mirrored parts in h-bridges.
Connections:
- net +5V: now also Q1.S, Q2.S, Q4.S, Q6.S; no longer Q1.D, Q2.D, Q4.D, Q6.D
- net N$1: now also Q1.D; no longer Q1.S
- net N$11: now also Q6.D; no longer Q6.S
- net N$12: now also Q2.D; no longer Q2.S
- net N$6: now also Q4.D; no longer Q4.S
Other:
- moved on the sheet: Q1, Q2, Q3, Q4, Q6

Commit message: updated schematics
* added molex-spox 3 pin connector library (for connecting to ax12a
servos
* updated schematic to fix 12v rail issue
* added datasheets
Parts:
- added U$2: AX-12A, molex-spox:AX-12A
- added X1: MKS1853-6-0-303, con-stocko:MKS1853-6-0-303
Connections:
- removed net +5V: Q1.S, Q2.S, Q4.S, Q6.S, R12.2, R13.2, R4.2, R5.2, R8.2, R9.2
- removed net N$5: D1.A, JP1.1
- new net 12V: D1.A, JP1.1, Q1.S, Q2.S, Q4.S, Q6.S, R12.2, R13.2, R4.2, R5.2, R8.2, R9.2, U$2.VDD
- net +HEIGHT: now also U$1.GPIO2_25
- net +RADIUS: now also U$1.GPIO2_23
- net -HEIGHT: now also U$1.GPIO2_24
- net -RADIUS: now also U$1.GPIO2_22
- net BBB_EQEP1A: now also U$1.UART4_CTSN
- net BBB_EQEP1B: now also U$1.UART4_RTSN
- net BBB_EQEP2A: now also U$1.GPIO1_12
- net BBB_EQEP2B: now also U$1.GPIO1_13
- net BBB_RX: now also U$1.UART1_RXD, U$1.UART2_RXD
- net BBB_TX: now also U$1.UART1_TXD, U$1.UART2_TXD
- net GND: now also U$2.GND
- net SERVO_TX/RX: now also U$2.DATA
Other:
- moved on the sheet: Q1, Q2, Q3, Q4, Q6, Q7, Q8, R-AXIS, Z-AXIS
