File: design/schematics/ArmControl/AGSE_BBB_cape.sch (EAGLE design)
At the start: 59 parts, among them Q1 PFET-FQP27P06, Q2 PFET-FQP27P06, Q3 NFET-FQP30N06L, Q4 NFET-FQP30N06L, Q5 PFET-FQP27P06, Q6 PFET-FQP27P06, Q7 NFET-FQP30N06L, Q8 NFET-FQP30N06L, U1 V_REG_LD1085D2

Commit message: Finalized schematic and board
also added pngs for reference.
Other:
- note added: "A"
- note added: "This schematic encompasses the electrical design of the AGSE motor control board. These circuits meet the following goals: 1. Vertical DC linear actuator motor control 2. Radial DC linear actuator motor control 3. Encoder Feedback for vertical motor encoder 4. Encoder Feedback for radial motor encoder 5. 12 V to 5 V power regulation for BeagleBone Black 6. Serial Buffer for controlling daisychain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"
- note added: "Vanderbilt Aerospace Club : AGSE Motor Control Board"
- note added: "William Emfinger"
- note removed: "This schematic encompasses the electrical design of the AGSE Radial and Height motor control circuits These electronics meet the following goals: (*) Motor actuation to increase and decrease the radial and height positions of the AGSE gripper"
- note removed: "Vanderbilt Aerospace Club : AGSE Linear Actuator Motor Controller"
Changed lines of the file:
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@@
 <sheet>
 <plain>
-<text x="-58.42" y="187.96" size="6.4516" layer="91">Vanderbilt Aerospace Club : AGSE
-Linear Actuator Motor Controller</text>
-<text x="-30.48" y="160.02" size="2.54" layer="91">This schematic encompasses the electrical design of
-the AGSE Radial and Height motor control circuits
-These electronics meet the following goals:
-(*) Motor actuation to increase and decrease the radial
-and height positions of the AGSE gripper</text>
+<text x="-58.42" y="187.96" size="6.4516" layer="91">Vanderbilt Aerospace Club :
+AGSE Motor Control Board</text>
+<text x="-58.42" y="182.88" size="3.81" layer="91" align="top-left">This schematic encompasses the electrical design of
+the AGSE motor control board.  These circuits meet the following goals:
+1. Vertical DC linear actuator motor control
+2. Radial DC linear actuator motor control
+3. Encoder Feedback for vertical motor encoder
+4. Encoder Feedback for radial motor encoder
+5. 12 V to 5 V power regulation for BeagleBone Black
+6. Serial Buffer for controlling daisychained servos:
+     * Main gripper servo motor
+     * Gripper wrist rotation servo motor
+     * AGSE arm base rotation servo motor
+This board mounts as a cape on the BeagleBone Black,
+providing it power and handling the associated
+connections for motor feedback and control.</text>
+<text x="-43.18" y="-60.96" size="5.08" layer="94">William Emfinger</text>
+<text x="33.02" y="-60.96" size="3.81" layer="94">A</text>
 </plain>
 <instances>
