File: design/schematics/ArmControl/AGSE_BBB_cape.brd (EAGLE design)
At the start: 71.8 x 54.6 mm, 55 parts, among them Q1 PFET-FQP27P06, Q2 PFET-FQP27P06, Q3 NFET-FQP30N06L, Q4 PFET-FQP27P06, Q5 NFET-FQP30N06L, Q6 PFET-FQP27P06, Q7 NFET-FQP30N06L, Q8 NFET-FQP30N06L, T1 2N2222, T2 2N2222, T3 2N2222, T4 2N2222, T5 2N3904, T6 2N3904, U1 V_REG_LD1085D2

Commit message: updated schematic symbols for h-bridges
Connections:
- net +5V: now also Q1.2, Q6.2; no longer Q1.3, Q6.3
- net GND: now also Q3.3, Q7.3; no longer Q3.2, Q7.2
- net N$1: now also Q1.3, Q3.2; no longer Q1.2, Q3.3
- net N$11: now also Q6.3, Q7.2; no longer Q6.2, Q7.3
Changed lines of the file:
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@@
 </polygon>
 <contactref element="Q5" pad="3"/>
-<contactref element="Q3" pad="2"/>
 <contactref element="T1" pad="1"/>
 <contactref element="T2" pad="1"/>
 <contactref element="Q8" pad="3"/>
-<contactref element="Q7" pad="2"/>
 <contactref element="T3" pad="1"/>
 <contactref element="T4" pad="1"/>
@@
 <contactref element="R23" pad="1"/>
 <contactref element="R22" pad="1"/>
+<contactref element="Q7" pad="3"/>
+<contactref element="Q3" pad="3"/>
 <wire x1="-43.815" y1="-83.947" x2="-43.815" y2="-88.265" width="0" layer="19" extent="1-1"/>
 <wire x1="-43.815" y1="-79.629" x2="-43.815" y2="-83.947" width="0" layer="19" extent="1-1"/>
@@
 <wire x1="-11.049" y1="-48.514" x2="-15.24" y2="-56.261" width="0" layer="19" extent="1-1"/>
 <wire x1="-2.413" y1="-56.261" x2="-11.049" y2="-48.514" width="0" layer="19" extent="1-1"/>
-<wire x1="-21.463" y1="-31.369" x2="-25.146" y2="-48.514" width="0" layer="19" extent="1-1"/>
-<wire x1="-14.732" y1="-18.415" x2="-21.463" y2="-31.369" width="0" layer="19" extent="1-1"/>
-<wire x1="-37.211" y1="-31.369" x2="-21.463" y2="-31.369" width="0" layer="19" extent="1-1"/>
-<wire x1="-0.635" y1="-31.369" x2="-14.732" y2="-18.415" width="0" layer="19" extent="1-1"/>
-<wire x1="21.59" y1="4.445" x2="-0.635" y2="-31.369" width="0" layer="19" extent="1-1"/>
+<wire x1="-18.923" y1="-31.369" x2="-25.146" y2="-48.514" width="0" layer="19" extent="1-1"/>
+<wire x1="-12.192" y1="-18.415" x2="-18.923" y2="-31.369" width="0" layer="19" extent="1-1"/>
+<wire x1="-0.635" y1="-31.369" x2="-12.192" y2="-18.415" width="0" layer="19" extent="1-1"/>
+<wire x1="-37.211" y1="-31.369" x2="-18.923" y2="-31.369" width="0" layer="19" extent="1-1"/>
+<wire x1="21.59" y1="4.445" x2="-12.192" y2="-18.415" width="0" layer="19" extent="1-1"/>
 <wire x1="21.59" y1="6.985" x2="21.59" y2="4.445" width="0" layer="19" extent="1-1"/>
 <wire x1="26.67" y1="13.01" x2="21.59" y2="6.985" width="0" layer="19" extent="1-1"/>
@@
 <signal name="+5V">
 <contactref element="Q4" pad="2"/>
-<contactref element="Q1" pad="3"/>
 <contactref element="R4" pad="2"/>
 <contactref element="R5" pad="2"/>
 <contactref element="Q2" pad="2"/>
-<contactref element="Q6" pad="3"/>
 <contactref element="R8" pad="2"/>
 <contactref element="R9" pad="2"/>
 <contactref element="R13" pad="2"/>
 <contactref element="R12" pad="2"/>
+<contactref element="Q6" pad="2"/>
+<contactref element="Q1" pad="2"/>
 <wire x1="-31.115" y1="-62.357" x2="-31.115" y2="-75.311" width="0" layer="19" extent="1-1"/>
-<wire x1="-37.211" y1="-49.403" x2="-31.115" y2="-62.357" width="0" layer="19" extent="1-1"/>
-<wire x1="-37.211" y1="-40.386" x2="-37.211" y2="-49.403" width="0" layer="19" extent="1-1"/>
-<wire x1="-22.733" y1="-40.386" x2="-37.211" y2="-40.386" width="0" layer="19" extent="1-1"/>
 <wire x1="-16.256" y1="-62.357" x2="-31.115" y2="-62.357" width="0" layer="19" extent="1-1"/>
 <wire x1="-16.256" y1="-66.675" x2="-16.256" y2="-62.357" width="0" layer="19" extent="1-1"/>
 <wire x1="-1.397" y1="-66.675" x2="-16.256" y2="-66.675" width="0" layer="19" extent="1-1"/>
 <wire x1="-1.397" y1="-70.993" x2="-1.397" y2="-66.675" width="0" layer="19" extent="1-1"/>
+<wire x1="-39.751" y1="-49.403" x2="-31.115" y2="-62.357" width="0" layer="19" extent="1-1"/>
+<wire x1="-39.751" y1="-40.386" x2="-39.751" y2="-49.403" width="0" layer="19" extent="1-1"/>
+<wire x1="-22.733" y1="-40.386" x2="-39.751" y2="-40.386" width="0" layer="19" extent="1-1"/>
 <wire x1="-5.715" y1="-40.386" x2="-22.733" y2="-40.386" width="0" layer="19" extent="1-1"/>
 </signal>
 <signal name="N$1">
-<contactref element="Q1" pad="2"/>
-<contactref element="Q3" pad="3"/>
 <contactref element="Z-AXIS" pad="2"/>
-<wire x1="-39.751" y1="-40.386" x2="10.922" y2="28.377" width="0" layer="19" extent="1-1"/>
-<wire x1="-12.192" y1="-18.415" x2="-39.751" y2="-40.386" width="0" layer="19" extent="1-1"/>
+<contactref element="Q3" pad="2"/>
+<contactref element="Q1" pad="3"/>
+<wire x1="-14.732" y1="-18.415" x2="-37.211" y2="-40.386" width="0" layer="19" extent="1-1"/>
+<wire x1="10.922" y1="28.377" x2="-14.732" y2="-18.415" width="0" layer="19" extent="1-1"/>
 </signal>
 <signal name="N$7">
@@
 <signal name="N$8">
 <contactref element="R5" pad="1"/>
+<contactref element="T2" pad="3"/>
+<contactref element="Q3" pad="1"/>
 <contactref element="Q1" pad="1"/>
-<contactref element="Q3" pad="1"/>
-<contactref element="T2" pad="3"/>
 <wire x1="-42.291" y1="-40.386" x2="-28.956" y2="-62.357" width="0" layer="19" extent="1-1"/>
 <wire x1="-8.509" y1="-45.974" x2="-28.956" y2="-62.357" width="0" layer="19" extent="1-1"/>
@@
 </signal>
 <signal name="N$11">
-<contactref element="Q6" pad="2"/>
-<contactref element="Q7" pad="3"/>
 <contactref element="R-AXIS" pad="2"/>
-<wire x1="-39.751" y1="-49.403" x2="10.922" y2="37.14" width="0" layer="19" extent="1-1"/>
-<wire x1="-18.923" y1="-31.369" x2="-39.751" y2="-49.403" width="0" layer="19" extent="1-1"/>
+<contactref element="Q6" pad="3"/>
+<contactref element="Q7" pad="2"/>
+<wire x1="-21.463" y1="-31.369" x2="-37.211" y2="-49.403" width="0" layer="19" extent="1-1"/>
+<wire x1="10.922" y1="37.14" x2="-21.463" y2="-31.369" width="0" layer="19" extent="1-1"/>
 </signal>
 <signal name="N$12">
@@
 <signal name="N$14">
 <contactref element="R9" pad="1"/>
+<contactref element="T4" pad="3"/>
 <contactref element="Q6" pad="1"/>
 <contactref element="Q7" pad="1"/>
-<contactref element="T4" pad="3"/>
 <wire x1="-25.527" y1="-54.991" x2="-42.291" y2="-49.403" width="0" layer="19" extent="1-1"/>
 <wire x1="-14.097" y1="-66.675" x2="-25.527" y2="-54.991" width="0" layer="19" extent="1-1"/>

Commit message: fixed mirrored parts in h-bridges.
Connections:
- net +5V: now also Q1.3, Q2.3, Q4.3, Q6.3; no longer Q1.2, Q2.2, Q4.2, Q6.2
- net N$1: now also Q1.2; no longer Q1.3
- net N$11: now also Q6.2; no longer Q6.3
- net N$12: now also Q2.2; no longer Q2.3
- net N$6: now also Q4.2; no longer Q4.3
Changed lines of the file:
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@@
 <contactref element="R23" pad="1"/>
 <contactref element="R22" pad="1"/>
+<contactref element="Q3" pad="3"/>
 <contactref element="Q7" pad="3"/>
-<contactref element="Q3" pad="3"/>
 <wire x1="-43.815" y1="-83.947" x2="-43.815" y2="-88.265" width="0" layer="19" extent="1-1"/>
 <wire x1="-43.815" y1="-79.629" x2="-43.815" y2="-83.947" width="0" layer="19" extent="1-1"/>
@@
 </signal>
 <signal name="+5V">
-<contactref element="Q4" pad="2"/>
+<contactref element="Q1" pad="3"/>
 <contactref element="R4" pad="2"/>
 <contactref element="R5" pad="2"/>
-<contactref element="Q2" pad="2"/>
+<contactref element="Q6" pad="3"/>
 <contactref element="R8" pad="2"/>
 <contactref element="R9" pad="2"/>
 <contactref element="R13" pad="2"/>
 <contactref element="R12" pad="2"/>
-<contactref element="Q6" pad="2"/>
-<contactref element="Q1" pad="2"/>
+<contactref element="Q4" pad="3"/>
+<contactref element="Q2" pad="3"/>
 <wire x1="-31.115" y1="-62.357" x2="-31.115" y2="-75.311" width="0" layer="19" extent="1-1"/>
+<wire x1="-37.211" y1="-49.403" x2="-31.115" y2="-62.357" width="0" layer="19" extent="1-1"/>
+<wire x1="-37.211" y1="-40.386" x2="-37.211" y2="-49.403" width="0" layer="19" extent="1-1"/>
 <wire x1="-16.256" y1="-62.357" x2="-31.115" y2="-62.357" width="0" layer="19" extent="1-1"/>
 <wire x1="-16.256" y1="-66.675" x2="-16.256" y2="-62.357" width="0" layer="19" extent="1-1"/>
 <wire x1="-1.397" y1="-66.675" x2="-16.256" y2="-66.675" width="0" layer="19" extent="1-1"/>
 <wire x1="-1.397" y1="-70.993" x2="-1.397" y2="-66.675" width="0" layer="19" extent="1-1"/>
-<wire x1="-39.751" y1="-49.403" x2="-31.115" y2="-62.357" width="0" layer="19" extent="1-1"/>
-<wire x1="-39.751" y1="-40.386" x2="-39.751" y2="-49.403" width="0" layer="19" extent="1-1"/>
-<wire x1="-22.733" y1="-40.386" x2="-39.751" y2="-40.386" width="0" layer="19" extent="1-1"/>
-<wire x1="-5.715" y1="-40.386" x2="-22.733" y2="-40.386" width="0" layer="19" extent="1-1"/>
+<wire x1="-20.193" y1="-40.386" x2="-37.211" y2="-40.386" width="0" layer="19" extent="1-1"/>
+<wire x1="-3.175" y1="-40.386" x2="-20.193" y2="-40.386" width="0" layer="19" extent="1-1"/>
 </signal>
 <signal name="N$1">
+<contactref element="Q1" pad="2"/>
 <contactref element="Z-AXIS" pad="2"/>
 <contactref element="Q3" pad="2"/>
-<contactref element="Q1" pad="3"/>
-<wire x1="-14.732" y1="-18.415" x2="-37.211" y2="-40.386" width="0" layer="19" extent="1-1"/>
+<wire x1="-14.732" y1="-18.415" x2="-39.751" y2="-40.386" width="0" layer="19" extent="1-1"/>
 <wire x1="10.922" y1="28.377" x2="-14.732" y2="-18.415" width="0" layer="19" extent="1-1"/>
 </signal>
 <signal name="N$7">
 <contactref element="R4" pad="1"/>
-<contactref element="Q4" pad="1"/>
 <contactref element="Q5" pad="1"/>
 <contactref element="T1" pad="3"/>
+<contactref element="Q4" pad="1"/>
 <wire x1="-22.606" y1="-45.974" x2="-43.815" y2="-62.357" width="0" layer="19" extent="1-1"/>
 <wire x1="-8.255" y1="-40.386" x2="-22.606" y2="-45.974" width="0" layer="19" extent="1-1"/>
@@
 <signal name="N$8">
 <contactref element="R5" pad="1"/>
+<contactref element="Q1" pad="1"/>
 <contactref element="T2" pad="3"/>
 <contactref element="Q3" pad="1"/>
-<contactref element="Q1" pad="1"/>
 <wire x1="-42.291" y1="-40.386" x2="-28.956" y2="-62.357" width="0" layer="19" extent="1-1"/>
 <wire x1="-8.509" y1="-45.974" x2="-28.956" y2="-62.357" width="0" layer="19" extent="1-1"/>
@@
 </signal>
 <signal name="N$11">
+<contactref element="Q6" pad="2"/>
 <contactref element="R-AXIS" pad="2"/>
-<contactref element="Q6" pad="3"/>
 <contactref element="Q7" pad="2"/>
-<wire x1="-21.463" y1="-31.369" x2="-37.211" y2="-49.403" width="0" layer="19" extent="1-1"/>
+<wire x1="-21.463" y1="-31.369" x2="-39.751" y2="-49.403" width="0" layer="19" extent="1-1"/>
 <wire x1="10.922" y1="37.14" x2="-21.463" y2="-31.369" width="0" layer="19" extent="1-1"/>
 </signal>
 <signal name="N$12">
 <contactref element="Q8" pad="2"/>
-<contactref element="Q2" pad="3"/>
 <contactref element="R-AXIS" pad="1"/>
-<wire x1="-20.193" y1="-40.386" x2="10.922" y2="40.64" width="0" layer="19" extent="1-1"/>
-<wire x1="-3.175" y1="-31.369" x2="-20.193" y2="-40.386" width="0" layer="19" extent="1-1"/>
+<contactref element="Q2" pad="2"/>
+<wire x1="-3.175" y1="-31.369" x2="-22.733" y2="-40.386" width="0" layer="19" extent="1-1"/>
+<wire x1="10.922" y1="40.64" x2="-3.175" y2="-31.369" width="0" layer="19" extent="1-1"/>
 </signal>
 <signal name="N$13">
 <contactref element="R8" pad="1"/>
-<contactref element="Q2" pad="1"/>
 <contactref element="Q8" pad="1"/>
 <contactref element="T3" pad="3"/>
+<contactref element="Q2" pad="1"/>
 <wire x1="-39.624" y1="-54.991" x2="-28.956" y2="-66.675" width="0" layer="19" extent="1-1"/>
 <wire x1="-25.273" y1="-40.386" x2="-39.624" y2="-54.991" width="0" layer="19" extent="1-1"/>
@@
 <signal name="N$14">
 <contactref element="R9" pad="1"/>
+<contactref element="Q6" pad="1"/>
 <contactref element="T4" pad="3"/>
-<contactref element="Q6" pad="1"/>
 <contactref element="Q7" pad="1"/>
 <wire x1="-25.527" y1="-54.991" x2="-42.291" y2="-49.403" width="0" layer="19" extent="1-1"/>
@@
 </signal>
 <signal name="N$6">
-<contactref element="Q4" pad="3"/>
 <contactref element="Q5" pad="2"/>
 <contactref element="Z-AXIS" pad="1"/>
-<wire x1="-39.751" y1="-31.369" x2="10.922" y2="31.877" width="0" layer="19" extent="1-1"/>
-<wire x1="-3.175" y1="-40.386" x2="-39.751" y2="-31.369" width="0" layer="19" extent="1-1"/>
+<contactref element="Q4" pad="2"/>
+<wire x1="-5.715" y1="-40.386" x2="-39.751" y2="-31.369" width="0" layer="19" extent="1-1"/>
+<wire x1="10.922" y1="31.877" x2="-5.715" y2="-40.386" width="0" layer="19" extent="1-1"/>
 </signal>
 </signals>

Commit message: updated schematics
* added molex-spox 3 pin connector library (for connecting to ax12a
servos
* updated schematic to fix 12v rail issue
* added datasheets
Parts:
- added U$2: AX-12A, molex-spox:SPOX-3
- added X1: MKS1853-6-0-303, con-stocko:MKS1853-6-0-303
Connections:
- removed net +5V: Q1.3, Q2.3, Q4.3, Q6.3, R12.2, R13.2, R4.2, R5.2, R8.2, R9.2
- removed net N$5: D1.A, JP1.1
- new net 12V: D1.A, JP1.1, Q1.3, Q2.3, Q4.3, Q6.3, R12.2, R13.2, R4.2, R5.2, R8.2, R9.2, U$2.P$2
- net +HEIGHT: now also U$1.30
- net +RADIUS: now also U$1.29
- net -HEIGHT: now also U$1.28
- net -RADIUS: now also U$1.27
- net BBB_EQEP1A: now also U$1.35
- net BBB_EQEP1B: now also U$1.33
- net BBB_EQEP2A: now also U$1.12
- net BBB_EQEP2B: now also U$1.11
- net BBB_RX: now also U$1.68, U$1.72
- net BBB_TX: now also U$1.67, U$1.70
- net GND: now also U$2.P$3
- net SERVO_TX/RX: now also U$2.P$1
Routing:
- net N$5: track 19.8 -> 0.00 mm
- net 12V: track 0.00 -> 19.8 mm

Commit message: working on board layout
Parts:
- removed D3: GREEN, SparkFun-LED:LED-0603
- removed JP2: M023.5MM, SparkFun-Connectors:SCREWTERMINAL-3.5MM-2
- removed R3: 510, SparkFun-Passives:0402-RES
- removed U$2: AX-12A, molex-spox:SPOX-3
- removed X1: MKS1853-6-0-303, con-stocko:MKS1853-6-0-303
- added SERVO: AX-12A, molex-spox:SPOX-3
- Q4: value PFET-FQP27P06 -> NFET-FQP30N06L
- Q5: value NFET-FQP30N06L -> PFET-FQP27P06
- R10, R11, R12, R13, R14, R15, R16, R17, R18, R19, R20, R21, R22, R23, R24, R4, R5, R6, R7, R8, R9: device resistor:0207/12 -> resistor:0204V
- T1, T2, T3, T4: value 2N2222 -> 2N3904; device transistor:TO18 -> transistor:TO92
- moved R10 150.4 mm to (70.6, 33.5), turned to 90 degrees
- moved R11 141.7 mm to (73.0, 33.5), turned to 270 degrees
- moved T3 138.7 mm to (65.0, 33.3), turned to 180 degrees
- moved Q1 134.7 mm to (62.6, 47.1), turned to 180 degrees
- moved T5 131.1 mm to (73.3, 41.5)
- moved T6 127.9 mm to (73.3, 47.8), turned to 180 degrees
- moved R4 125.7 mm to (24.3, 47.1), turned to 90 degrees
- moved R8 125.0 mm to (51.7, 33.9)
- moved T4 123.9 mm to (65.0, 26.9)
- moved R7 121.3 mm to (25.8, 36.8), turned to 270 degrees
- moved R9 119.4 mm to (56.6, 33.9), turned to 180 degrees
- moved R5 117.6 mm to (20.3, 47.1), turned to 90 degrees
- moved Q6 117.5 mm to (38.2, 38.5)
- moved Q2 116.2 mm to (62.6, 38.5)
- moved Q5 110.6 mm to (38.2, 47.1), turned to 180 degrees
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Connections:
- removed net N$2: D3.C, R3.2
- net 12V: now also Q5.3, SERVO.P$2; no longer Q4.3, U$2.P$2
- net 5V: no longer D3.A, JP2.1
- net GND: now also Q4.3, SERVO.P$3, T1.3, T2.3, T3.3, T4.3; no longer JP2.2, Q5.3, R3.1, T1.1, T2.1, T3.1, T4.1, U$2.P$3
- net N$1: now also Q6.2, Q8.2; no longer Q1.2, Q3.2
- net N$11: now also Q2.2, Q4.2; no longer Q6.2, Q7.2
- net N$12: now also Q1.2, Q3.2; no longer Q2.2, Q8.2
- net N$13: now also Q1.1, Q3.1, T3.1; no longer Q2.1, Q8.1, T3.3
- net N$14: now also Q2.1, Q4.1, T4.1; no longer Q6.1, Q7.1, T4.3
- net N$6: now also Q7.2; no longer Q4.2
- net N$7: now also Q7.1, T1.1; no longer Q4.1, T1.3
- net N$8: now also Q6.1, Q8.1, T2.1; no longer Q1.1, Q3.1, T2.3
- net SERVO_TX/RX: now also SERVO.P$1; no longer U$2.P$1
Routing:
- net 5V: track 32.4 -> 5.71 mm
- net 12V: track 19.8 -> 14.9 mm
- net VOUT: track 50.2 -> 47.5 mm
- net N$2: track 2.28 -> 0.00 mm
Other:
- board text added: "12V"
- board text removed: "12 VDC IN"
- board text removed: "5 VDC Regulated"
